File: AE-7SEG-BOARD.kicad_pcb (KiCad board)
At the start: 2 copper layers, 12 x 25.5 mm, 16 parts, among them U1 74HC595D, 118, U2 7-SEGMENT-LED

Commit message: Add files via upload
Parts:
- C1, R1, R10, R11, R2, R3, R4, R5, R6, R7, R8, R9, U1: moved to B.Cu
- CH1, CH2: value Conn_01x05_Female -> Conn_01x05_Male; footprint Connector_PinSocket_2.54mm:PinSocket_1x05_P2.54mm_Vertical -> Connector_PinHeader_2.54mm:PinHeader_1x05_P2.54mm_Vertical
- U2: moved to F.Cu
- moved CH2 60.8 mm to (95.2, 82.5), turned to -90 degrees
- moved U2 60.8 mm to (95.2, 78.7)
- moved CH1 60.8 mm to (95.2, 59.7), turned to -90 degrees
- moved C1 59.9 mm to (95.9, 66.0)
- moved R8 58.2 mm to (97.2, 76.2)
- moved R9 58.2 mm to (97.2, 66.0)
- moved R7 56.5 mm to (98.4, 76.2)
- moved R10 54.9 mm to (99.7, 66.0)
- moved R6 54.9 mm to (99.7, 76.2)
- moved U1 54.1 mm to (100.3, 71.1)
- moved R11 53.3 mm to (101.0, 66.0)
- moved R5 53.3 mm to (101.0, 76.2)
- moved R4 51.9 mm to (102.2, 76.2)
- moved R1 50.5 mm to (103.5, 66.0)
- moved R3 50.5 mm to (103.5, 76.2)
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