File: AE-7SEG-BOARD.kicad_pcb (KiCad board)
At the start: 2 copper layers, 12 x 25.5 mm, 16 parts, among them U1 74HC595D, 118, U2 7-SEGMENT-LED

Commit message: Add files via upload
Parts:
- C1, CH1, CH2, R1, R10, R11, R2, R3, R4, R5, R6, R7, R8, R9, U1: moved to F.Cu
- U2: moved to B.Cu
- moved CH1 80.5 mm to (162.4, 104.1)
- moved CH2 80.5 mm to (162.4, 127.0)
- moved U2 80.5 mm to (162.4, 123.2)
- moved C1 79.5 mm to (161.8, 110.5)
- moved R8 77.4 mm to (160.5, 120.7)
- moved R9 77.4 mm to (160.5, 110.5)
- moved R7 75.3 mm to (159.2, 120.7)
- moved R10 73.3 mm to (158.0, 110.5)
- moved R6 73.3 mm to (158.0, 120.7)
- moved U1 72.3 mm to (157.3, 115.6)
- moved R11 71.3 mm to (156.7, 110.5)
- moved R5 71.3 mm to (156.7, 120.7)
- moved R4 69.3 mm to (155.4, 120.7)
- moved R3 67.4 mm to (154.2, 120.7)
- moved R1 67.4 mm to (154.2, 110.5)
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