File: AE-7SEG-BOARD.kicad_sch (KiCad schematic)
At the start: 16 parts, among them U1 74HC595D, 118, U2 7-SEGMENT-LED

Commit message: Add files via upload
Parts:
- removed CH1, CH2: Conn_01x05_Female, Connector_PinSocket_2.54mm:PinSocket_1x05_P2.54mm_Vertical, symbol Connector:Conn_01x05_Female
- added CH1, CH2: Conn_01x05_Male, Connector_PinHeader_2.54mm:PinHeader_1x05_P2.54mm_Vertical, symbol Connector:Conn_01x05_Male
Connections:
- net GND: now also CH1.2 (Pin_2), CH2.5 (Pin_5)
- net LATCH: now also CH2.2 (Pin_2)
- net MR#: now also CH2.1 (Pin_1)
- net OE: now also CH2.3 (Pin_3)
- net SCK: now also CH1.3 (Pin_3)
- net SDI: now also CH1.4 (Pin_4)
- net SDO: now also CH1.5 (Pin_5)
- net VCC: now also CH1.1 (Pin_1), CH2.4 (Pin_4)
Other:
- title: (none) -> AE-7SEG-BOARD
- moved on the sheet: C1, R1, R10, R11, R2, R3, R4, R5, R6, R7, R8, R9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

Commit message: Add files via upload
Parts:
- CH1, CH2, U2: now left out of the parts list
Other:
- moved on the sheet: C1, CH1, CH2, R1, R10, R11, R2, R3, R4, R5, R6, R7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

Commit message: Add files via upload
Parts:
- U1: JLCPCB Rotation Offset (none) -> -90
Changed lines of the file:
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@@
   (junction (at 106.68 110.49) (diameter 0) (color 0 0 0 0)
   )
-  (junction (at 147.32 113.03) (diameter 0) (color 0 0 0 0)
-  )
   (junction (at 147.32 72.39) (diameter 0) (color 0 0 0 0)
   )
@@
     (stroke (width 0) (type default))
   )
-  (wire (pts (xy 147.32 114.3) (xy 147.32 113.03))
-    (stroke (width 0) (type default))
-  )
-  (wire (pts (xy 144.78 113.03) (xy 147.32 113.03))
+  (wire (pts (xy 147.32 111.76) (xy 147.32 114.3))
     (stroke (width 0) (type default))
   )
@@
     (stroke (width 0) (type default))
   )
-  (wire (pts (xy 147.32 113.03) (xy 147.32 111.76))
-    (stroke (width 0) (type default))
-  )
   (wire (pts (xy 157.48 106.68) (xy 160.02 106.68))
     (stroke (width 0) (type default))
@@
   )
   (wire (pts (xy 180.34 99.06) (xy 172.72 99.06))
-    (stroke (width 0) (type default))
-  )
-  (wire (pts (xy 147.32 72.39) (xy 149.86 72.39))
     (stroke (width 0) (type default))
   )
@@
     )
   )
-  (symbol (lib_id "power:PWR_FLAG") (at 149.86 72.39 270) (unit 1)
-    (in_bom yes) (on_board yes) (dnp no) (fields_autoplaced)
-    (property "Reference" "#FLG0101" (at 151.765 72.39 0)
-      (effects (font (size 1.27 1.27)) hide)
-    )
-    (property "Value" "PWR_FLAG" (at 153.67 72.3899 90)
-      (effects (font (size 1.27 1.27)) (justify left))
-    )
-    (property "Footprint" "" (at 149.86 72.39 0)
-      (effects (font (size 1.27 1.27)) hide)
-    )
-    (property "Datasheet" "~" (at 149.86 72.39 0)
-      (effects (font (size 1.27 1.27)) hide)
-    )
-    (pin "1")
-    (instances
-      (project "AE-7SEG-BOARD"
-        (path "/38975fd9-2a31-4e73-b8fb-7891ecf7d40d"
-          (reference "#FLG0101") (unit 1)
-        )
-      )
-    )
-  )
   (symbol (lib_id "power:VCC") (at 101.6 102.87 270) (unit 1)
     (in_bom yes) (on_board yes) (dnp no)
@@
     )
     (property "LCSC" "C5947" (at 147.32 93.98 0)
+      (effects (font (size 1.27 1.27)) hide)
+    )
+    (property "JLCPCB Rotation Offset" "-90" (at 147.32 93.98 0)
       (effects (font (size 1.27 1.27)) hide)
     )
@@
         )
       )
-    )
-  )
-  (symbol (lib_id "power:PWR_FLAG") (at 144.78 113.03 90) (unit 1)
-    (in_bom yes) (on_board yes) (dnp no) (fields_autoplaced)
-    (property "Reference" "#FLG0102" (at 142.875 113.03 0)
-      (effects (font (size 1.27 1.27)) hide)
-    )
-    (property "Value" "PWR_FLAG" (at 140.97 113.0299 90)
-      (effects (font (size 1.27 1.27)) (justify left))
-    )
-    (property "Footprint" "" (at 144.78 113.03 0)
-      (effects (font (size 1.27 1.27)) hide)
-    )
-    (property "Datasheet" "~" (at 144.78 113.03 0)
-      (effects (font (size 1.27 1.27)) hide)
-    )
-    (pin "1")
-    (instances
-      (project "AE-7SEG-BOARD"
-        (path "/38975fd9-2a31-4e73-b8fb-7891ecf7d40d"
-          (reference "#FLG0102") (unit 1)
-        )
-      )
